Commit message: frame update

File: robotshyu/robots/NRMK/indy7/indy7_description/indy7_frame.urdf (robot description, URDF)
Before this commit: robot indy7, 8 links, 7 joints
Links:
- link link0: geometry 
- link link1: geometry 
- link link2: geometry 
- link link3: geometry 
- link link4: geometry 
- link link5: geometry 
- link link6: geometry 
- link tcp: geometry visual mesh filename=meshes/frame/untitled.obj scale=0.05 0.05 0.05

File: robotshyu/robots/NRMK/indyrp2/indyrp2_description/indyrp2_frame.urdf (robot description, URDF)
Before this commit: robot indyrp2, 10 links, 9 joints
Links:
- link link0: geometry 
- link link1: geometry 
- link link2: geometry 
- link link3: geometry 
- link link4: geometry 
- link link5: geometry 
- link link6: geometry 
- link link7: geometry 
- link tcp: geometry visual mesh filename=meshes/frame/untitled.obj scale=0.05 0.05 0.05
