Commit message: NRMK model update

File: robotshyu/robots/NRMK/indy7/indy7_description/indy7.urdf (robot description, URDF)
Before this commit: robot indy7, 8 links, 7 joints
Links:
- link link0: mass 1.59306955 -> 1.67030785; geometry visual mesh filename=meshes/stl/Indy7_0.stl
- link link1: mass 11.8030102 -> 11.44444535; geometry visual mesh filename=meshes/stl/Indy7_1.stl
- link link2: mass 7.99292141 -> 5.84766553; geometry visual mesh filename=meshes/stl/Indy7_2.stl
- link link3: mass 2.99134127 -> 2.68206064; geometry visual mesh filename=meshes/stl/Indy7_3.stl
- link link4: mass 2.12317035 -> 2.12987371; geometry visual mesh filename=meshes/stl/Indy7_4.stl
- link link5: mass 2.28865091 -> 2.22412271; geometry visual mesh filename=meshes/stl/Indy7_5.stl
- link link6: mass 0.40083918 -> 0.38254932; geometry visual mesh filename=meshes/stl/Indy7_6.stl

File: robotshyu/robots/NRMK/indy7/indy7_description/indy7_frame.urdf (robot description, URDF)
Before this commit: robot indy7, 8 links, 7 joints
Links:
- link link0: mass 1.59306955 -> 1.67030785
- link link1: mass 11.8030102 -> 11.44444535
- link link2: mass 7.99292141 -> 5.84766553
- link link3: mass 2.99134127 -> 2.68206064
- link link4: mass 2.12317035 -> 2.12987371
- link link5: mass 2.28865091 -> 2.22412271
- link link6: mass 0.40083918 -> 0.38254932

File: robotshyu/robots/NRMK/indyrp2/indyrp2_description/indyrp2.urdf (robot description, URDF)
Before this commit: robot indyrp2, 10 links, 9 joints
Links:
- removed link world
- link link0: mass 5.44309 -> 1.67030785; geometry visual mesh filename=meshes/stl/IndyRP2_0.stl
- link link1: mass 5.50328 -> 11.44444535; geometry visual mesh filename=meshes/stl/IndyRP2_1.stl
- link link2: mass 5.95397 -> 4.43308185; geometry visual mesh filename=meshes/stl/IndyRP2_2.stl
- link link3: mass 4.08259 -> 2.87045928; geometry visual mesh filename=meshes/stl/IndyRP2_3.stl
- link link4: mass 4.02733 -> 2.68206064; geometry visual mesh filename=meshes/stl/IndyRP2_4.stl
- link link5: mass 2.52863 -> 2.12987371; geometry visual mesh filename=meshes/stl/IndyRP2_5.stl
- link link6: mass 2.03152 -> 2.22412271; geometry visual mesh filename=meshes/stl/IndyRP2_6.stl
- link link7: mass 0.17194 -> 0.38254932; geometry visual mesh filename=meshes/stl/IndyRP2_7.stl
Joints:
- removed joint global

File: robotshyu/robots/NRMK/indyrp2/indyrp2_description/indyrp2_frame.urdf (robot description, URDF)
Before this commit: robot indyrp2, 10 links, 9 joints
Links:
- removed link world
- link link0: mass 5.44309 -> 1.67030785
- link link1: mass 5.50328 -> 11.44444535
- link link2: mass 5.95397 -> 4.43308185
- link link3: mass 4.08259 -> 2.87045928
- link link4: mass 4.02733 -> 2.68206064
- link link5: mass 2.52863 -> 2.12987371
- link link6: mass 2.03152 -> 2.22412271
- link link7: mass 0.17194 -> 0.38254932
Joints:
- removed joint global

Commit message: tcp update

File: robotshyu/robots/NRMK/indy7/indy7_description/indy7.urdf (robot description, URDF)
Before this commit: robot indy7, 8 links, 7 joints
Joints:
- joint indy7_tcp: origin xyz=0 0 0.06 rpy=0 0 0 -> xyz=0 0 0.23 rpy=0 0 0

File: robotshyu/robots/NRMK/indy7/indy7_description/indy7_frame.urdf (robot description, URDF)
Before this commit: robot indy7, 8 links, 7 joints
Joints:
- joint indy7_tcp: origin xyz=0 0 0.06 rpy=0 0 0 -> xyz=0 0 0.23 rpy=0 0 0

Commit message: update

File: robotshyu/robots/NRMK/indy7/indy7_description/indy7.urdf (robot description, URDF)
Before this commit: robot indy7, 8 links, 7 joints
Joints:
- joint indy7_tcp: origin xyz=0 0 0.23 rpy=0 0 0 -> xyz=0 0 0.0795 rpy=0 0 0
