Commit message: hyumm update

File: robotshyu/robots/NRMK/indy7/indy7_description/indy7_nom.urdf (robot description, URDF)
Before this commit: robot indy7, 8 links, 7 joints
Links:
- link link0: geometry visual mesh filename=meshes/stl/Indy7_0.stl
- link link1: geometry visual mesh filename=meshes/stl/Indy7_1.stl
- link link2: geometry visual mesh filename=meshes/stl/Indy7_2.stl
- link link3: geometry visual mesh filename=meshes/stl/Indy7_3.stl
- link link4: geometry visual mesh filename=meshes/stl/Indy7_4.stl
- link link5: geometry visual mesh filename=meshes/stl/Indy7_5.stl
- link link6: geometry visual mesh filename=meshes/stl/Indy7_6.stl
