Commit message: update: task limit

File: robotshyu/robots/mir250/description/mir250_ppr.urdf (robot description, URDF)
Before this commit: robot mir250_ppr, 6 links, 5 joints
Links:
- link base_link: geometry visual mesh filename=meshes/visual/mir_250_base.stl scale=1 1 1

Commit message: Update MiR250 URDF

File: robotshyu/robots/mir250/description/mir250_ppr.urdf (robot description, URDF)
Before this commit: robot mir250_ppr, 6 links, 5 joints
Links:
- removed link base_footprint
- added link back_laser_link, mass 1.2; visual mesh filename=meshes/visual/sick_lms-100.stl
- added link bl_caster_rotation_link, mass 0.3097539019; visual mesh filename=meshes/visual/caster_wheel_base.stl
- added link bl_caster_wheel_link, mass 1.0; visual cylinder length=0.032 radius=0.0625
- added link br_caster_rotation_link, mass 0.3097539019; visual mesh filename=meshes/visual/caster_wheel_base.stl
- added link br_caster_wheel_link, mass 1.0; visual cylinder length=0.032 radius=0.0625
- added link fl_caster_rotation_link, mass 0.3097539019; visual mesh filename=meshes/visual/caster_wheel_base.stl
- added link fl_caster_wheel_link, mass 1.0; visual cylinder length=0.032 radius=0.0625
- added link fr_caster_rotation_link, mass 0.3097539019; visual mesh filename=meshes/visual/caster_wheel_base.stl
- added link fr_caster_wheel_link, mass 1.0; visual cylinder length=0.032 radius=0.0625
- added link front_laser_link, mass 1.2; visual mesh filename=meshes/visual/sick_lms-100.stl
- added link imu_frame, mass 0.000001
- added link imu_link, mass 0.000001
- added link left_wheel_link, mass 1.0; visual cylinder length=0.038 radius=0.1
- added link right_wheel_link, mass 1.0; visual cylinder length=0.038 radius=0.1
- added link us_1_frame, mass 0.000001
- added link us_2_frame, mass 0.000001
- link base_link: mass 58.0 -> 97.0; geometry collision box size=0.8 0.58 0.615; visual mesh filename=meshes/visual/mir_250_base.stl
Joints:
- removed joint base_joint
- added joint base_link_to_back_laser_joint: type fixed, parent base_link, child back_laser_link, origin xyz=-0.319485 -0.205 0.1914 rpy=0.0 0.0 -2.356194490192345
- added joint base_link_to_front_laser_joint: type fixed, parent base_link, child front_laser_link, origin xyz=0.310515 0.205 0.1914 rpy=0.0 0.0 0.7853981633974483
- added joint base_link_to_imu_joint: type fixed, parent base_link, child imu_link, origin xyz=0.0 0.0 0.25 rpy=0 0 0
- added joint bl_caster_rotation_joint: type fixed, parent base_link, child bl_caster_rotation_link, origin xyz=-0.300485 0.188 0.1565 rpy=0 0 0, axis 0 0 1
- added joint bl_caster_wheel_joint: type fixed, parent bl_caster_rotation_link, child bl_caster_wheel_link, origin xyz=-0.0382 0 -0.094 rpy=0 0 0, axis 0 1 0
- added joint br_caster_rotation_joint: type fixed, parent base_link, child br_caster_rotation_link, origin xyz=-0.300485 -0.188 0.1565 rpy=0 0 0, axis 0 0 1
- added joint br_caster_wheel_joint: type fixed, parent br_caster_rotation_link, child br_caster_wheel_link, origin xyz=-0.0382 0 -0.094 rpy=0 0 0, axis 0 1 0
- added joint fl_caster_rotation_joint: type fixed, parent base_link, child fl_caster_rotation_link, origin xyz=0.299215 0.188 0.1565 rpy=0 0 0, axis 0 0 1
- added joint fl_caster_wheel_joint: type fixed, parent fl_caster_rotation_link, child fl_caster_wheel_link, origin xyz=-0.0382 0 -0.094 rpy=0 0 0, axis 0 1 0
- added joint fr_caster_rotation_joint: type fixed, parent base_link, child fr_caster_rotation_link, origin xyz=0.299215 -0.188 0.1565 rpy=0 0 0, axis 0 0 1
- added joint fr_caster_wheel_joint: type fixed, parent fr_caster_rotation_link, child fr_caster_wheel_link, origin xyz=-0.0382 0 -0.094 rpy=0 0 0, axis 0 1 0
- added joint imu_link_to_imu_frame_joint: type fixed, parent imu_link, child imu_frame, origin xyz=0 0 0 rpy=0 0 0
- added joint left_wheel_joint: type fixed, parent base_link, child left_wheel_link, origin xyz=0.0 0.2015 0.1 rpy=0 0 0, axis 0 1 0, limit effort=100 velocity=20.0
- added joint right_wheel_joint: type fixed, parent base_link, child right_wheel_link, origin xyz=0.0 -0.2015 0.1 rpy=0 0 0, axis 0 1 0, limit effort=100 velocity=20.0
- added joint us_1_joint: type fixed, parent base_link, child us_1_frame, origin xyz=0.45 -0.12 0.16  rpy=0 0 0
- added joint us_2_joint: type fixed, parent base_link, child us_2_frame, origin xyz=0.45 0.12 0.16  rpy=0 0 0
- joint lin_x_joint: limit lower=-1e+16 upper=1e+16 effort=1000.0 velocity=1.5 -> lower=-1e+16 upper=1e+16 effort=1000.0 velocity=3.5
- joint lin_y_joint: limit lower=-1e+16 upper=1e+16 effort=1000.0 velocity=1.5 -> lower=-1e+16 upper=1e+16 effort=1000.0 velocity=3.5
- joint rot_z_joint: limit lower=-1e+16 upper=1e+16 effort=1000.0 velocity=0.7 -> lower=-1e+16 upper=1e+16 effort=1000.0 velocity=3.5

File: robotshyu/robots/mir250/description/mir250_ppr_frame.urdf (robot description, URDF)
Before this commit: robot mir250_ppr, 6 links, 5 joints
Links:
- removed link base_footprint
- added link back_laser_link, mass 1.2
- added link bl_caster_rotation_link, mass 0.3097539019
- added link bl_caster_wheel_link, mass 1.0
- added link br_caster_rotation_link, mass 0.3097539019
- added link br_caster_wheel_link, mass 1.0
- added link fl_caster_rotation_link, mass 0.3097539019
- added link fl_caster_wheel_link, mass 1.0
- added link fr_caster_rotation_link, mass 0.3097539019
- added link fr_caster_wheel_link, mass 1.0
- added link front_laser_link, mass 1.2
- added link imu_frame, mass 0.000001
- added link imu_link, mass 0.000001
- added link left_wheel_link, mass 1.0
- added link right_wheel_link, mass 1.0
- added link us_1_frame, mass 0.000001
- added link us_2_frame, mass 0.000001
- link base_link: mass 58.0 -> 97.0
Joints:
- removed joint base_joint
- added joint base_link_to_back_laser_joint: type fixed, parent base_link, child back_laser_link, origin xyz=-0.319485 -0.205 0.1914 rpy=0.0 0.0 -2.356194490192345
- added joint base_link_to_front_laser_joint: type fixed, parent base_link, child front_laser_link, origin xyz=0.310515 0.205 0.1914 rpy=0.0 0.0 0.7853981633974483
- added joint base_link_to_imu_joint: type fixed, parent base_link, child imu_link, origin xyz=0.0 0.0 0.25 rpy=0 0 0
- added joint bl_caster_rotation_joint: type fixed, parent base_link, child bl_caster_rotation_link, origin xyz=-0.300485 0.188 0.1565 rpy=0 0 0, axis 0 0 1
- added joint bl_caster_wheel_joint: type fixed, parent bl_caster_rotation_link, child bl_caster_wheel_link, origin xyz=-0.0382 0 -0.094 rpy=0 0 0, axis 0 1 0
- added joint br_caster_rotation_joint: type fixed, parent base_link, child br_caster_rotation_link, origin xyz=-0.300485 -0.188 0.1565 rpy=0 0 0, axis 0 0 1
- added joint br_caster_wheel_joint: type fixed, parent br_caster_rotation_link, child br_caster_wheel_link, origin xyz=-0.0382 0 -0.094 rpy=0 0 0, axis 0 1 0
- added joint fl_caster_rotation_joint: type fixed, parent base_link, child fl_caster_rotation_link, origin xyz=0.299215 0.188 0.1565 rpy=0 0 0, axis 0 0 1
- added joint fl_caster_wheel_joint: type fixed, parent fl_caster_rotation_link, child fl_caster_wheel_link, origin xyz=-0.0382 0 -0.094 rpy=0 0 0, axis 0 1 0
- added joint fr_caster_rotation_joint: type fixed, parent base_link, child fr_caster_rotation_link, origin xyz=0.299215 -0.188 0.1565 rpy=0 0 0, axis 0 0 1
- added joint fr_caster_wheel_joint: type fixed, parent fr_caster_rotation_link, child fr_caster_wheel_link, origin xyz=-0.0382 0 -0.094 rpy=0 0 0, axis 0 1 0
- added joint imu_link_to_imu_frame_joint: type fixed, parent imu_link, child imu_frame, origin xyz=0 0 0 rpy=0 0 0
- added joint left_wheel_joint: type fixed, parent base_link, child left_wheel_link, origin xyz=0.0 0.2015 0.1 rpy=0 0 0, axis 0 1 0, limit effort=100 velocity=20.0
- added joint right_wheel_joint: type fixed, parent base_link, child right_wheel_link, origin xyz=0.0 -0.2015 0.1 rpy=0 0 0, axis 0 1 0, limit effort=100 velocity=20.0
- added joint us_1_joint: type fixed, parent base_link, child us_1_frame, origin xyz=0.45 -0.12 0.16  rpy=0 0 0
- added joint us_2_joint: type fixed, parent base_link, child us_2_frame, origin xyz=0.45 0.12 0.16  rpy=0 0 0
- joint lin_x_joint: limit lower=-1e+16 upper=1e+16 effort=1000.0 velocity=1.5 -> lower=-1e+16 upper=1e+16 effort=1000.0 velocity=3.5
- joint lin_y_joint: limit lower=-1e+16 upper=1e+16 effort=1000.0 velocity=1.5 -> lower=-1e+16 upper=1e+16 effort=1000.0 velocity=3.5
- joint rot_z_joint: limit lower=-1e+16 upper=1e+16 effort=1000.0 velocity=0.7 -> lower=-1e+16 upper=1e+16 effort=1000.0 velocity=3.5

File: robotshyu/robots/turtlebot3/description/turtlebot3_burger_frame.urdf (robot description, URDF)
Before this commit: robot turtlebot3_burger, 10 links, 9 joints
Links:
- link base_link: geometry visual mesh filename=meshes/frame/untitled.obj scale=0.05 0.05 0.05
