Commit message: indyrp gravity

File: robotshyu/robots/NRMK/indyrp2/indyrp2_description/indyrp2.urdf (robot description, URDF)
Before this commit: robot indyrp2, 9 links, 8 joints
Joints:
- joint joint0: limit (none) -> lower=-3.0543261909900763 upper=3.0543261909900763 effort=10 velocity=1; type continuous -> revolute
- joint joint1: limit (none) -> lower=-3.0543261909900763 upper=3.0543261909900763 effort=10 velocity=1; type continuous -> revolute
- joint joint2: limit (none) -> lower=-3.0543261909900763 upper=3.0543261909900763 effort=10 velocity=1; type continuous -> revolute
- joint joint3: limit (none) -> lower=-3.0543261909900763 upper=3.0543261909900763 effort=10 velocity=1; type continuous -> revolute
- joint joint4: limit (none) -> lower=-3.0543261909900763 upper=3.0543261909900763 effort=10 velocity=1; type continuous -> revolute
- joint joint5: limit (none) -> lower=-3.0543261909900763 upper=3.0543261909900763 effort=10 velocity=1; type continuous -> revolute
- joint joint6: limit (none) -> lower=-3.0543261909900763 upper=3.0543261909900763 effort=10 velocity=1; type continuous -> revolute
