Commit message: update

File: robotshyu/robots/HYUMOB/hyumob_description/hyumob.urdf (robot description, URDF)
Before this commit: robot hyumob, 8 links, 7 joints
Links:
- removed link wheel_left_back
- removed link wheel_left_front
- removed link wheel_right_back
- removed link wheel_right_front
- link base_link: mass 50.03647319 -> 53.53736408
Joints:
- removed joint joint_left_back
- removed joint joint_left_front
- removed joint joint_right_back
- removed joint joint_right_front
