Commit message: update

File: robotshyu/robots/HYUMM/hyumm_description/hyumm_floating.urdf (robot description, URDF)
Before this commit: robot hyumm, 12 links, 11 joints
Links:
- removed link lin_x_link
- removed link lin_y_link
- link tcp: mass 0 -> 0.000001
- link world: mass 0 -> 0.000001
Joints:
- removed joint lin_x_joint
- removed joint lin_y_joint
- removed joint rot_z_joint
- added joint base_world: type fixed, parent world, child base_link, origin xyz=0.0 0 0.0 rpy=0 0 0

File: robotshyu/robots/HYUMM/hyumm_description/hyumm_multi.urdf (robot description, URDF)
Before this commit: robot hyumm, 12 links, 11 joints
Links:
- removed link base_link
- removed link link0
- removed link link1
- removed link link2
- removed link link3
- removed link link4
- removed link link5
- removed link link6
- removed link tcp
- added link base_center, mass 0
- added link l_base_link, mass 53.53736408; collision mesh filename=meshes/stl/base_link.STL; visual mesh filename=meshes/stl/base_link.STL
- added link l_link0, mass 1.67030785; visual mesh filename=meshes/stl/Indy7_0.stl
- added link l_link1, mass 11.44444535; visual mesh filename=meshes/stl/Indy7_1.stl
- added link l_link2, mass 5.84766553; visual mesh filename=meshes/stl/Indy7_2.stl
- added link l_link3, mass 2.68206064; visual mesh filename=meshes/stl/Indy7_3.stl
- added link l_link4, mass 2.12987371; visual mesh filename=meshes/stl/Indy7_4.stl
- added link l_link5, mass 2.22412271; visual mesh filename=meshes/stl/Indy7_5.stl
- added link l_link6, mass 0.38254932; visual mesh filename=meshes/stl/Indy7_6.stl
- added link l_tcp, mass 0
- added link r_base_link, mass 53.53736408; collision mesh filename=meshes/stl/base_link.STL; visual mesh filename=meshes/stl/base_link.STL
- added link r_link0, mass 1.67030785; visual mesh filename=meshes/stl/Indy7_0.stl
- added link r_link1, mass 11.44444535; visual mesh filename=meshes/stl/Indy7_1.stl
- added link r_link2, mass 5.84766553; visual mesh filename=meshes/stl/Indy7_2.stl
- added link r_link3, mass 2.68206064; visual mesh filename=meshes/stl/Indy7_3.stl
- added link r_link4, mass 2.12987371; visual mesh filename=meshes/stl/Indy7_4.stl
- added link r_link5, mass 2.22412271; visual mesh filename=meshes/stl/Indy7_5.stl
- added link r_link6, mass 0.38254932; visual mesh filename=meshes/stl/Indy7_6.stl
- added link r_tcp, mass 0
Joints:
- removed joint base_flange
- removed joint indy7_tcp
- removed joint joint0
- removed joint joint1
- removed joint joint2
- removed joint joint3
- removed joint joint4
- removed joint joint5
- added joint l_base_flange: type fixed, parent l_base_link, child l_link0, origin xyz=0.3 0 0.228 rpy=0 0 0
- added joint l_base_joint: type fixed, parent base_center, child l_base_link, origin xyz=0 0.4 0.0 rpy=0 0 0
- added joint l_indy7_tcp: type fixed, parent l_link6, child l_tcp, origin xyz=0 0 0.23 rpy=0 0 0
- added joint l_joint0: type revolute, parent l_link0, child l_link1, origin xyz=0 0 0.0775 rpy=0 0 0, axis 0 0 1, limit lower=-3.0543261909900763 upper=3.0543261909900763 effort=10 velocity=1
- added joint l_joint1: type revolute, parent l_link1, child l_link2, origin xyz=0 -0.10900000 0.22200000 rpy=1.5707963267948966 1.5707963267948966 0, axis 0 0 1, limit lower=-3.0543261909900763 upper=3.0543261909900763 effort=10 velocity=1
- added joint l_joint2: type revolute, parent l_link2, child l_link3, origin xyz=-0.45000000 +0.00000000 -0.03050000 rpy=0 0 0, axis 0 0 1, limit lower=-3.0543261909900763 upper=3.0543261909900763 effort=10 velocity=1
- added joint l_joint3: type revolute, parent l_link3, child l_link4, origin xyz=-0.26700000 +0.00000000 -0.07500000 rpy=-1.5707963267948966 0 1.5707963267948966, axis 0 0 1, limit lower=-3.0543261909900763 upper=3.0543261909900763 effort=10 velocity=1
- added joint l_joint4: type revolute, parent l_link4, child l_link5, origin xyz=+0.00000000 -0.11400000 +0.08300000 rpy=1.5707963267948966 1.5707963267948966 0, axis 0 0 1, limit lower=-3.0543261909900763 upper=3.0543261909900763 effort=10 velocity=1
- added joint l_joint5: type revolute, parent l_link5, child l_link6, origin xyz=-0.16800000 +0.00000000 +0.06900000 rpy=-1.5707963267948966 0 1.5707963267948966, axis 0 0 1, limit lower=-3.752457891787808 upper=3.752457891787808 effort=10 velocity=1
- added joint r_base_flange: type fixed, parent r_base_link, child r_link0, origin xyz=0.3 0 0.228 rpy=0 0 0
- added joint r_base_joint: type fixed, parent base_center, child r_base_link, origin xyz=0 -0.4 0.0 rpy=0 0 0
- added joint r_indy7_tcp: type fixed, parent r_link6, child r_tcp, origin xyz=0 0 0.23 rpy=0 0 0
- added joint r_joint0: type revolute, parent r_link0, child r_link1, origin xyz=0 0 0.0775 rpy=0 0 0, axis 0 0 1, limit lower=-3.0543261909900763 upper=3.0543261909900763 effort=10 velocity=1
- added joint r_joint1: type revolute, parent r_link1, child r_link2, origin xyz=0 -0.10900000 0.22200000 rpy=1.5707963267948966 1.5707963267948966 0, axis 0 0 1, limit lower=-3.0543261909900763 upper=3.0543261909900763 effort=10 velocity=1
- added joint r_joint2: type revolute, parent r_link2, child r_link3, origin xyz=-0.45000000 +0.00000000 -0.03050000 rpy=0 0 0, axis 0 0 1, limit lower=-3.0543261909900763 upper=3.0543261909900763 effort=10 velocity=1
- added joint r_joint3: type revolute, parent r_link3, child r_link4, origin xyz=-0.26700000 +0.00000000 -0.07500000 rpy=-1.5707963267948966 0 1.5707963267948966, axis 0 0 1, limit lower=-3.0543261909900763 upper=3.0543261909900763 effort=10 velocity=1
- added joint r_joint4: type revolute, parent r_link4, child r_link5, origin xyz=+0.00000000 -0.11400000 +0.08300000 rpy=1.5707963267948966 1.5707963267948966 0, axis 0 0 1, limit lower=-3.0543261909900763 upper=3.0543261909900763 effort=10 velocity=1
- added joint r_joint5: type revolute, parent r_link5, child r_link6, origin xyz=-0.16800000 +0.00000000 +0.06900000 rpy=-1.5707963267948966 0 1.5707963267948966, axis 0 0 1, limit lower=-3.752457891787808 upper=3.752457891787808 effort=10 velocity=1
- joint rot_z_joint: child base_link -> base_center

File: robotshyu/robots/HYUMM/hyumm_description/hyumm_offset.urdf (robot description, URDF)
Before this commit: robot hyumm, 12 links, 11 joints
Links:
- link lin_x_link: mass 0 -> 0.000001
- link lin_y_link: mass 0 -> 0.000001
- link tcp: mass 0 -> 0.000001
- link world: mass 0 -> 0.000001
Joints:
- joint lin_x_joint: origin xyz=0 0 0 rpy=0 0 0 -> xyz=0 0.4 0 rpy=0 0 0

File: robotshyu/robots/HYUMM/hyumm_description/hyumm_offset_l.urdf (robot description, URDF)
Before this commit: robot hyumm, 12 links, 11 joints
Links:
- added link base_center, mass 0
Joints:
- added joint base_joint: type fixed, parent base_center, child base_link, origin xyz=0 0.4 0.0 rpy=0 0 0
- joint rot_z_joint: child base_link -> base_center

File: robotshyu/robots/HYUMM/hyumm_description/hyumm_offset_r.urdf (robot description, URDF)
Before this commit: robot hyumm, 12 links, 11 joints
Links:
- added link base_center, mass 0
Joints:
- added joint base_joint: type fixed, parent base_center, child base_link, origin xyz=0 -0.4 0.0 rpy=0 0 0
- joint rot_z_joint: child base_link -> base_center
