Commit message: hyumm

File: robotshyu/robots/HYUMM/hyumm_description/hyumm.urdf (robot description, URDF)
Before this commit: robot hyumm, 13 links, 12 joints
Links:
- added link lin_x_link, mass 0.000001
- added link lin_y_link, mass 0.000001
- added link world, mass 0.000001
Joints:
- added joint lin_x_joint: type prismatic, parent world, child lin_x_link, origin xyz=0 0 0 rpy=0 0 0, axis 1 0 0, limit lower=-1e+16 upper=1e+16 effort=1000.0 velocity=3.5
- added joint lin_y_joint: type prismatic, parent lin_x_link, child lin_y_link, origin xyz=0 0 0 rpy=0 0 0, axis 0 1 0, limit lower=-1e+16 upper=1e+16 effort=1000.0 velocity=3.5
- added joint rot_z_joint: type revolute, parent lin_y_link, child base_link, origin xyz=0 0 0 rpy=0 0 0, axis 0 0 1, limit lower=-1e+16 upper=1e+16 effort=1000.0 velocity=3.5
- joint base_flange: origin xyz=0.3 0 0.198 rpy=0 0 0 -> xyz=0.3 0 0.228 rpy=0 0 0
- joint joint_left_back: axis 0 -1 0 -> (none); limit lower=0 upper=0 effort=0 velocity=0 -> (none); origin xyz=-0.41 -0.269 0.05 rpy=0 0 0 -> xyz=-0.41 -0.269 0.08 rpy=0 0 0
- joint joint_left_front: axis 0 -1 0 -> (none); limit lower=0 upper=0 effort=0 velocity=0 -> (none); origin xyz=0.41 -0.269 0.05 rpy=0 0 0 -> xyz=0.41 -0.269 0.08 rpy=0 0 0
- joint joint_right_back: axis 0 -1 0 -> (none); limit lower=0 upper=0 effort=0 velocity=0 -> (none); origin xyz=-0.41 0.269 0.05 rpy=0 0 0 -> xyz=-0.41 0.269 0.08 rpy=0 0 0
- joint joint_right_front: axis 0 -1 0 -> (none); limit lower=0 upper=0 effort=0 velocity=0 -> (none); origin xyz=0.41 0.269 0.05 rpy=0 0 0 -> xyz=0.41 0.269 0.08 rpy=0 0 0

Commit message: indy7, hyumm inertia update

File: robotshyu/robots/HYUMM/hyumm_description/hyumm.urdf (robot description, URDF)
Before this commit: robot hyumm, 16 links, 15 joints
Joints:
- joint indy7_tcp: origin xyz=0 0 0.06 rpy=0 0 0 -> xyz=0 0 0.23 rpy=0 0 0

Commit message: update

File: robotshyu/robots/HYUMM/hyumm_description/hyumm.urdf (robot description, URDF)
Before this commit: robot hyumm, 12 links, 11 joints
Links:
- link tcp: geometry collision box size=0.1 0.1 0.1; visual box size=0.1 0.1 0.1

File: robotshyu/robots/HYUMM/hyumm_description/hyumm_nom.urdf (robot description, URDF)
Before this commit: robot hyumm_nom, 12 links, 11 joints
Links:
- link base_link: geometry visual mesh filename=meshes/stl/base_link.STL

File: robotshyu/robots/KUKA/kr250_rail/description/kuka_kr_250_rail_nom.urdf (robot description, URDF)
Before this commit: robot kuka_kr_250_rail, 12 links, 11 joints
Links:
- link FTSensor: geometry visual mesh filename=meshes/ft_sensor.stl

File: robotshyu/robots/NRMK/indy7/indy7_description/indy7.urdf (robot description, URDF)
Before this commit: robot indy7, 8 links, 7 joints
Links:
- link tcp: geometry collision box size=0.1 0.1 0.1; visual box size=0.1 0.1 0.1
