Commit message: update

File: robotshyu/robots/KUKA/kr120/kr120_description/kuka_kr_120.urdf (robot description, URDF)
Before this commit: robot kuka_kr_120, 9 links, 8 joints
Joints:
- joint tcp_joint: origin xyz=0.0 0.0 -0.02 rpy=-1.57079632679 0.0 -1.57079632679 -> xyz=0.0 0.0 -0.02 rpy=3.1415926536 0.0 1.5707963268

File: robotshyu/robots/KUKA/kr120/kr120_description/kuka_kr_120_frame.urdf (robot description, URDF)
Before this commit: robot kuka_kr_120, 9 links, 8 joints
Joints:
- joint tcp_joint: origin xyz=0.0 0.0 -0.02 rpy=-1.57079632679 0.0 -1.57079632679 -> xyz=0.0 0.0 -0.02 rpy=3.1415926536 0.0 1.5707963268
