Commit message: update

File: robotshyu/robots/HYUSPA/hyu_spa_description/hyu_spa.urdf (robot description, URDF)
Before this commit: robot hyu_spa, 8 links, 7 joints
Links:
- added link link7, mass 0.59063954; visual mesh filename=meshes/stl/hyu_spa_7.stl
Joints:
- added joint joint6: type revolute, parent link6, child link7, origin xyz=0 0 -0.084 rpy=0 0 0, axis 0 1 0, limit lower=-3.752457891787808 upper=3.752457891787808 effort=10 velocity=1
- joint tcp_fixed: parent link6 -> link7
