Commit message: update

File: robotshyu/robots/HDR/yl012/yl012_description/yl012_sat_core.urdf (robot description, URDF)
Before this commit: robot yl102_sat_core, 11 links, 10 joints
Links:
- added link link_flange, mass 0.71; collision mesh filename=meshes/link_FT.stl; visual mesh filename=meshes/link_FT.stl
- added link link_tcp_CoM, mass 00
- link link_ft: mass 0.71 -> 00; geometry 
Joints:
- added joint flange_fixed: type fixed, parent link6, child link_flange, origin xyz=0 0 0.07385 rpy=0 0 0, axis 0 0 0
- added joint tcp_CoM_fixed: type fixed, parent link_ft, child link_tcp_CoM, origin xyz=-0.00001166 -0.00000932 0.13976902 rpy=0 0 0, axis 0 0 0
- joint core_fixed: origin xyz=0 0 0.0412 rpy=0 0 0 -> xyz=0.00001166 0.00000932 -0.12976902 rpy=0 0 0; parent link_ft -> link_tcp_CoM
- joint ft_fixed: origin xyz=0 0 0.07385 rpy=0 0 0 -> xyz=0 0 0.0312 rpy=0 0 0; parent link6 -> link_flange

Commit message: update

File: robotshyu/robots/HDR/yl012/yl012_description/yl012_sat_core.urdf (robot description, URDF)
Before this commit: robot yl102_sat_core, 13 links, 12 joints
Joints:
- joint core_fixed: origin xyz=0.00001166 0.00000932 -0.12976902 rpy=0 0 0 -> xyz=0 0 0.01 rpy=0 0 0; parent link_tcp_CoM -> link_ft
- joint tcp_CoM_fixed: origin xyz=-0.00001166 -0.00000932 0.13976902 rpy=0 0 0 -> xyz=-0.00001166 -0.00000932 -0.04673098 rpy=0 0 0; parent link_ft -> link_sat
