Commit message: update

File: robotshyu/robots/KARM/KARM_EM/KARM_EM_description/KARM_EM.urdf (robot description, URDF)
Before this commit: robot KARM_EM, 10 links, 9 joints
Links:
- link ASM_LINK_0_EM: mass 0.47278619   -> 0.47278619; geometry collision mesh filename=../meshes/ASM_LINK_0_EM.STL; visual mesh filename=../meshes/ASM_LINK_0_EM.STL
- link ASM_LINK_1_EM: geometry collision mesh filename=../meshes/ASM_LINK_1_EM.STL; visual mesh filename=../meshes/ASM_LINK_1_EM.STL
- link ASM_LINK_2_EM: mass 1.08543372   -> 1.08543372; geometry collision mesh filename=../meshes/ASM_LINK_2_EM.STL; visual mesh filename=../meshes/ASM_LINK_2_EM.STL
- link ASM_LINK_3_EM: geometry collision mesh filename=../meshes/ASM_LINK_3_EM.STL; visual mesh filename=../meshes/ASM_LINK_3_EM.STL
- link ASM_LINK_4_EM: geometry collision mesh filename=../meshes/ASM_LINK_4_EM.STL; visual mesh filename=../meshes/ASM_LINK_4_EM.STL
- link ASM_LINK_5_EM: mass 8.50980173  -> 8.50980173; geometry collision mesh filename=../meshes/ASM_LINK_5_EM.STL; visual mesh filename=../meshes/ASM_LINK_5_EM.STL
- link ASM_LINK_6_EM: geometry collision mesh filename=../meshes/ASM_LINK_6_EM.STL; visual mesh filename=../meshes/ASM_LINK_6_EM.STL
- link ASM_LINK_7_EM: mass 0.47459064  -> 0.47459064; geometry collision mesh filename=../meshes/ASM_LINK_7_EM.STL; visual mesh filename=../meshes/ASM_LINK_7_EM.STL

Commit message: update: EQM_V2

File: robotshyu/robots/KARM/KARM_EM/KARM_EM_description/KARM_EM.urdf (robot description, URDF)
Before this commit: robot KARM_EM, 10 links, 9 joints
Links:
- link ASM_LINK_0_EM: geometry collision mesh filename=/meshes/ASM_LINK_0.STL; visual mesh filename=/meshes/ASM_LINK_0.STL
- link ASM_LINK_1_EM: geometry collision mesh filename=/meshes/ASM_LINK_1.STL; visual mesh filename=/meshes/ASM_LINK_1.STL
- link ASM_LINK_2_EM: geometry collision mesh filename=/meshes/ASM_LINK_2.STL; visual mesh filename=/meshes/ASM_LINK_2.STL
- link ASM_LINK_3_EM: geometry collision mesh filename=/meshes/ASM_LINK_3.STL; visual mesh filename=/meshes/ASM_LINK_3.STL
- link ASM_LINK_4_EM: geometry collision mesh filename=/meshes/ASM_LINK_4.STL; visual mesh filename=/meshes/ASM_LINK_4.STL
- link ASM_LINK_5_EM: geometry collision mesh filename=/meshes/ASM_LINK_5.STL; visual mesh filename=/meshes/ASM_LINK_5.STL
- link ASM_LINK_6_EM: geometry collision mesh filename=/meshes/ASM_LINK_6.STL; visual mesh filename=/meshes/ASM_LINK_6.STL
- link ASM_LINK_7_EM: geometry collision mesh filename=/meshes/ASM_LINK_7.STL; visual mesh filename=/meshes/ASM_LINK_7.STL

File: robotshyu/robots/KARM/KARM_EQM/KARM_EQM_description/KARM_EQM.urdf (robot description, URDF)
Before this commit: robot KARM_EQM, 10 links, 9 joints
Links:
- removed link eef_link
- removed link link0
- added link base_link, mass 2.7715; collision mesh filename=meshes/base_link.STL; visual mesh filename=meshes/base_link.STL
- added link tcp, mass 0.0
- link link1: mass 4.4336 -> 6.5395; geometry collision mesh filename=meshes/link1.STL; visual mesh filename=meshes/link1.STL
- link link2: mass 5.33597958831089 -> 14.5254250159894; geometry collision mesh filename=meshes/link2.STL; visual mesh filename=meshes/link2.STL
- link link3: mass 4.3966 -> 6.4825; geometry collision mesh filename=meshes/link3.STL; visual mesh filename=meshes/link3.STL
- link link4: mass 4.06563238726737 -> 5.77091277717193; geometry collision mesh filename=meshes/link4.STL; visual mesh filename=meshes/link4.STL
- link link5: mass 4.39661533299087 -> 13.5; geometry collision mesh filename=meshes/link5.STL; visual mesh filename=meshes/link5.STL
- link link6: mass 4.62888290048359 -> 6.53953654625201; geometry collision mesh filename=meshes/link6.STL; visual mesh filename=meshes/link6.STL
- link link7: mass 1.2654 -> 2.91241532737351; geometry collision mesh filename=meshes/link7.STL; visual mesh filename=meshes/link7.STL
Joints:
- removed joint eef_fixed
- added joint tcp_fixed: type fixed, parent link7, child tcp, origin xyz=0 0 0.083 rpy=0 0 0
- joint joint1: limit lower=-3.14 upper=3.14 effort=100 velocity=10 -> lower=-3.14 upper=3.14 effort=400 velocity=3.14; origin xyz=0 0 0.128 rpy=0 0 0 -> xyz=0 0 0.087 rpy=0 0 3.141592; parent link0 -> base_link
- joint joint2: axis 0 1 0 -> 0 0 1; limit lower=-3.14 upper=3.14 effort=100 velocity=10 -> lower=-3.14 upper=3.14 effort=400 velocity=3.14; origin xyz=0 0.0915 0.128 rpy=0 0 0 -> xyz=0 0.097 0.112 rpy=1.5708 -1.5708 0
- joint joint3: limit lower=-3.14 upper=3.14 effort=100 velocity=10 -> lower=-3.14 upper=3.14 effort=400 velocity=3.14; origin xyz=0 0.0915 1.0012 rpy=0 0.021863 0 -> xyz=0.988 0 -0.095 rpy=-1.5708 0 -1.5708
- joint joint4: axis 0 1 0 -> 0 0 -1; limit lower=-3.14 upper=3.14 effort=100 velocity=10 -> lower=-3.14 upper=3.14 effort=400 velocity=3.14; origin xyz=-0.009811 -0.0915 0.44867 rpy=0 -0.021863 0 -> xyz=0 -0.097 0.112 rpy=-1.5708 -1.5708 0
- joint joint5: limit lower=-3.14 upper=3.14 effort=100 velocity=10 -> lower=-3.14 upper=3.14 effort=400 velocity=3.14; origin xyz=0 -0.0915 0.6045 rpy=0 0 0 -> xyz=0.114 0 -0.095 rpy=1.5708 0 1.5708
- joint joint6: axis 0 1 0 -> 0 0 1; limit lower=-3.14 upper=3.14 effort=100 velocity=10 -> lower=-3.14 upper=3.14 effort=400 velocity=3.14; origin xyz=0 -0.0915 0.4455 rpy=0 0 0 -> xyz=0 -0.097 0.786 rpy=-1.5704 -1.5708 3.1412
- joint joint7: limit lower=-3.14 upper=3.14 effort=100 velocity=10 -> lower=-3.14 upper=3.14 effort=400 velocity=3.14; origin xyz=0 -0.0915 0.128 rpy=0 0 0 -> xyz=0.114 0 0.095 rpy=-1.5708 0 -1.5708
- joint world_fixed: axis (none) -> 0 0 1; child link0 -> base_link
