Commit message: update

File: robotshyu/robots/NRMK/indy12_v2_sat/description/indy12_v2_sat.urdf (robot description, URDF)
Before this commit: robot indy12_v2_sat, 22 links, 21 joints
Links:
- link tool_plange: mass 2.6 -> 0.300
Joints:
- joint Pz: limit lower=-2 upper=2 effort=10000 velocity=1000 -> lower=-1 upper=10 effort=10000 velocity=1000
- joint Rx: limit lower=-3.14 upper=3.14 effort=10000 velocity=1000 -> lower=-6.28 upper=6.28 effort=10000 velocity=1000
- joint Ry: limit lower=-3.14 upper=3.14 effort=10000 velocity=1000 -> lower=-6.28 upper=6.28 effort=10000 velocity=1000
- joint Rz: limit lower=-3.14 upper=3.14 effort=10000 velocity=1000 -> lower=-6.28 upper=6.28 effort=10000 velocity=1000
